Commit message: criada esqueleto de uma casa para teste e adicionado no mundo de teste

File: src/test_bot/models/mobile_bot.urdf (robot description, URDF)
Before this commit: robot mobile_bot, 4 links, 3 joints
Links:
- added link lidar_link, mass 0.114; collision cylinder length=0.18 radius=0.0508; visual cylinder length=0.18 radius=0.0508
Joints:
- added joint lidar_joint: type fixed, parent base_link, child lidar_link, origin xyz=0.215 0 0.13 rpy=0 0 0

Commit message: ajustado o laser lidar

File: src/test_bot/models/mobile_bot.urdf (robot description, URDF)
Before this commit: robot mobile_bot, 5 links, 4 joints
Links:
- link lidar_link: mass 0.114 -> 0.1; geometry collision cylinder length=0.04 radius=0.05; visual cylinder length=0.04 radius=0.05
